File: Design og implementering/Body HW/Proximity_sensor/Proximity_sensor_sch.brd (EAGLE design)
At the start: 77.3 x 55.9 mm, 11 parts, among them IC1 TINY26P, J1 RJ11-6PTH, J2 RJ11-6PTH, U2 LM2750SD-5.0

Commit message: Made final changes to eagle designs and exported to gerber -Felix
Routing:
- net GND: track 187.4 -> 191.2 mm
- net N$2: track 74.3 -> 77.2 mm
- net VCC: track 234.1 -> 232.3 mm
Changed lines of the file:
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@@
 </class>
 </classes>
-<designrules name="default">
+<designrules name="default *">
 <description language="de">&lt;b&gt;EAGLE Design Rules&lt;/b&gt;
 &lt;p&gt;
@@
 <param name="mdViaViaSameLayer" value="8mil"/>
 <param name="mnLayersViaInSmd" value="2"/>
-<param name="mdCopperDimension" value="40mil"/>
+<param name="mdCopperDimension" value="20mil"/>
 <param name="mdDrill" value="8mil"/>
 <param name="mdSmdStop" value="0mil"/>
@@
 <wire x1="38.1" y1="21.59" x2="34.925" y2="21.59" width="0.4064" layer="16"/>
 <wire x1="34.925" y1="21.59" x2="34.29" y2="20.955" width="0.4064" layer="16"/>
-<wire x1="46.99" y1="34.29" x2="46.99" y2="25.4" width="0.4064" layer="16"/>
-<wire x1="46.99" y1="34.29" x2="43.18" y2="34.29" width="0.4064" layer="16"/>
-<wire x1="43.18" y1="34.29" x2="43.18" y2="40.64" width="0.4064" layer="16"/>
-<wire x1="43.18" y1="40.64" x2="44.45" y2="41.91" width="0.4064" layer="16"/>
+<wire x1="46.99" y1="30.48" x2="46.99" y2="25.4" width="0.4064" layer="16"/>
 <wire x1="53.34" y1="63.5" x2="53.34" y2="62.23" width="0.4064" layer="16"/>
 <wire x1="53.34" y1="62.23" x2="57.15" y2="58.42" width="0.4064" layer="16"/>
@@
 <wire x1="40.64" y1="45.72" x2="44.45" y2="41.91" width="0.4064" layer="16"/>
 <wire x1="44.45" y1="48.26" x2="40.64" y2="48.26" width="0.4064" layer="16"/>
-<via x="60.833" y="25.4" extent="1-16" drill="0.6" shape="square"/>
-<via x="60.96" y="19.685" extent="1-16" drill="0.6" shape="square"/>
+<via x="60.833" y="25.4" extent="1-16" drill="0.6096" shape="square"/>
+<via x="60.96" y="19.685" extent="1-16" drill="0.6096" shape="square"/>
 <wire x1="60.96" y1="19.685" x2="60.96" y2="25.273" width="0.3048" layer="1"/>
 <wire x1="60.96" y1="25.273" x2="60.833" y2="25.4" width="0.3048" layer="1"/>
@@
 <wire x1="78.105" y1="32.385" x2="77.978" y2="32.385" width="0.4064" layer="16"/>
 <wire x1="77.978" y1="32.385" x2="77.978" y2="36.83" width="0.4064" layer="16"/>
+<wire x1="46.99" y1="34.29" x2="46.99" y2="30.48" width="0.4064" layer="16"/>
+<wire x1="46.99" y1="30.48" x2="43.18" y2="30.48" width="0.4064" layer="16"/>
+<wire x1="43.18" y1="30.48" x2="43.18" y2="39.37" width="0.4064" layer="16"/>
+<wire x1="43.18" y1="39.37" x2="44.45" y2="40.64" width="0.4064" layer="16"/>
+<wire x1="44.45" y1="40.64" x2="44.45" y2="41.91" width="0.4064" layer="16"/>
 </signal>
 <signal name="N$1">
@@
 <wire x1="27.94" y1="18.415" x2="31.75" y2="22.225" width="0.4064" layer="16"/>
 <wire x1="80.01" y1="18.415" x2="66.675" y2="18.415" width="0.4064" layer="16"/>
-<wire x1="44.45" y1="34.29" x2="44.45" y2="39.37" width="0.4064" layer="16"/>
-<wire x1="44.45" y1="39.37" x2="52.07" y2="39.37" width="0.4064" layer="16"/>
-<wire x1="52.07" y1="39.37" x2="53.34" y2="38.1" width="0.4064" layer="16"/>
 <wire x1="53.34" y1="38.1" x2="53.34" y2="30.48" width="0.4064" layer="16"/>
 <wire x1="53.34" y1="30.48" x2="67.31" y2="30.48" width="0.4064" layer="16"/>
@@
 <wire x1="79.5528" y1="32.131" x2="79.5528" y2="32.385" width="0.254" layer="16"/>
 <wire x1="72.136" y1="34.544" x2="71.12" y2="35.56" width="0.254" layer="16"/>
-<wire x1="81.915" y1="32.131" x2="81.915" y2="43.307" width="0.254" layer="1"/>
-<wire x1="81.915" y1="43.307" x2="82.042" y2="43.434" width="0.254" layer="1"/>
-<via x="82.042" y="43.434" extent="1-16" drill="0.5" diameter="0.6096" shape="square"/>
-<wire x1="82.042" y1="43.434" x2="88.9" y2="43.434" width="0.254" layer="16"/>
 <wire x1="88.9" y1="43.434" x2="89.408" y2="43.942" width="0.254" layer="16"/>
-<via x="81.915" y="32.131" extent="1-16" drill="0.5" diameter="0.6096" shape="square"/>
-<via x="81.915" y="29.718" extent="1-16" drill="0.5" diameter="0.6096" shape="square"/>
-<via x="78.359" y="29.718" extent="1-16" drill="0.5" diameter="0.6096" shape="square"/>
+<via x="81.915" y="32.131" extent="1-16" drill="0.6096" diameter="0.6096" shape="square"/>
+<via x="81.915" y="29.718" extent="1-16" drill="0.6096" diameter="0.6096" shape="square"/>
+<via x="78.359" y="29.718" extent="1-16" drill="0.6096" diameter="0.6096" shape="square"/>
 <wire x1="78.359" y1="29.718" x2="75.184" y2="29.718" width="0.254" layer="1"/>
-<via x="75.184" y="29.718" extent="1-16" drill="0.5" diameter="0.6096" shape="square"/>
+<via x="75.184" y="29.718" extent="1-16" drill="0.6096" diameter="0.6096" shape="square"/>
 <wire x1="75.184" y1="29.718" x2="74.295" y2="30.099" width="0.254" layer="16"/>
 <wire x1="74.295" y1="30.099" x2="72.009" y2="32.385" width="0.254" layer="16"/>
@@
 <wire x1="81.915" y1="32.131" x2="81.915" y2="29.718" width="0.3048" layer="1"/>
 <wire x1="78.359" y1="29.718" x2="81.915" y2="29.718" width="0.3048" layer="1"/>
+<wire x1="44.45" y1="34.29" x2="44.45" y2="38.1" width="0.4064" layer="16"/>
+<wire x1="44.45" y1="38.1" x2="53.34" y2="38.1" width="0.4064" layer="16"/>
+<wire x1="88.9" y1="43.434" x2="81.915" y2="43.434" width="0.254" layer="16"/>
+<via x="81.915" y="43.434" extent="1-16" drill="0.6096" shape="square"/>
+<wire x1="81.915" y1="43.434" x2="81.915" y2="32.131" width="0.254" layer="1"/>
 </signal>
 <signal name="N$2">
@@
 <wire x1="29.21" y1="15.24" x2="29.21" y2="17.145" width="0.4064" layer="16"/>
 <wire x1="29.21" y1="17.145" x2="31.75" y2="19.685" width="0.4064" layer="16"/>
-<wire x1="31.75" y1="19.685" x2="31.75" y2="20.32" width="0.4064" layer="16"/>
-<wire x1="31.75" y1="20.32" x2="33.02" y2="21.59" width="0.4064" layer="16"/>
-<wire x1="33.02" y1="21.59" x2="33.02" y2="33.02" width="0.4064" layer="16"/>
-<wire x1="33.02" y1="33.02" x2="34.29" y2="34.29" width="0.4064" layer="16"/>
+<wire x1="31.75" y1="19.685" x2="32.639" y2="21.209" width="0.254" layer="16"/>
+<wire x1="32.639" y1="21.209" x2="33.274" y2="21.844" width="0.254" layer="16"/>
+<wire x1="33.274" y1="21.844" x2="34.544" y2="22.225" width="0.254" layer="16"/>
+<wire x1="34.544" y1="22.225" x2="35.941" y2="22.606" width="0.254" layer="16"/>
+<wire x1="35.941" y1="22.606" x2="36.83" y2="23.495" width="0.254" layer="16"/>
+<wire x1="36.83" y1="23.495" x2="36.83" y2="30.48" width="0.254" layer="16"/>
+<wire x1="36.83" y1="30.48" x2="34.29" y2="33.02" width="0.254" layer="16"/>
+<wire x1="34.29" y1="33.02" x2="34.29" y2="34.29" width="0.254" layer="16"/>
 </signal>
 <signal name="N$3">
@@
 <wire x1="86.741" y1="33.909" x2="87.63" y2="33.02" width="0.3048" layer="16"/>
 </signal>
-<signal name="N$10">
-<via x="40.64" y="27.94" extent="1-16" drill="1" diameter="1.9304"/>
-</signal>
-<signal name="N$11">
-<via x="64.77" y="63.5" extent="1-16" drill="1" diameter="1.9304"/>
-</signal>
-<signal name="N$12">
-<via x="68.58" y="35.56" extent="1-16" drill="0.7" diameter="1.016" shape="square"/>
-</signal>
 <signal name="N$14">
 </signal>
@@
 </signal>
 <signal name="N$19">
-</signal>
-<signal name="N$20">
-<via x="81.915" y="32.131" extent="1-16" drill="0.5" diameter="0.6096" shape="square"/>
-</signal>
-<signal name="N$21">
-<via x="82.042" y="43.434" extent="1-16" drill="0.5" diameter="0.6096" shape="square"/>
 </signal>
 <signal name="N$25">
@@
 </signal>
 </signals>
+<errors>
+</errors>
 </board>
 </drawing>
